File: Hardware/esp32-thing.brd (EAGLE design)
At the start: 25.4 x 58.9 mm, 67 parts, among them Q1 2.5A/30V, Q2 MBT3904DW1T1, U1 MCP73831, U3 AP2112K-3.3V, U4 FT231XS, U5 W25Q32FVSS, Y1 26MHz, Y2 32.768kHz

Commit message: Incorporate changes from Jim's protos.
Parts:
- removed C1, C2: 270pF, SparkFun-Capacitors:0603-CAP
- added JP1, JP3: (no value), SparkFun-Passives:PAD-JUMPER-3-3OF3_NC_BY_TRACE_YES_SILK_FULL_BOX
- added R10, R11, R12, R9: 4.7K, SparkFun-Resistors:0603-RES
- added R15: 10K, SparkFun-Resistors:0603-RES@1
- J1, J2: device SparkFun-Connectors:1X20_NOSILK -> SparkFun-Connectors:MOLEX-1X4_LOCK
- R1, R13, R14, R3, R4, R6, R8: device SparkFun-Resistors:0603 -> SparkFun-Resistors:0603-RES
- U$1: value (none) -> ESP32
- moved J2 28.8 mm to (0.51, 17.8)
- moved J1 27.3 mm to (0.51, 28.6)
- moved C3 6.74 mm to (23.2, 33.4), turned to 90 degrees
- moved C18 5.62 mm to (17.8, 36.3)
- moved Y1 3.14 mm to (20.7, 33.4), turned to 180 degrees
- moved C17 1.91 mm to (12.7, 27.3)
- moved C5 1.89 mm to (17.8, 38.9)
- moved R2 1.89 mm to (17.8, 37.6)
- moved C23 1.54 mm to (17.0, 31.2), turned to 0 degrees
- moved C24 0.90 mm to (8.76, 30.1)
- moved R17 0.89 mm to (19.1, 18.2)
- moved C20 0.89 mm to (15.2, 40.4)
- moved C4 0.46 mm to (18.2, 33.4), turned to 270 degrees
- renumbered U2 to U$1
Connections:
- net N$11 renamed VCC_FLASH
- removed net 12: J1.8, U$1.18
- removed net 13: J1.7, U$1.20
- removed net 14: J1.9, U$1.17
- removed net 15: J2.11, U$1.21
- removed net 16: J2.6, U$1.26
- removed net 17: J2.7, U$1.27
- removed net 18: J2.13, U$1.35
- removed net 19: J2.20, U$1.41
- removed net 2: J2.10, U$1.22
- removed net 20: J2.19, U$1.40
- removed net 21: J2.18, U$1.39
- removed net 22: J2.17, U$1.38
- removed net 23: J2.14
- removed net 25: J1.12, U$1.14
- removed net 26: J1.11, U$1.15
- removed net 27: J1.10, U$1.16
- removed net 34: J1.14, U$1.10
- removed net 35: J1.13, U$1.11
- removed net 36: C1.2, J1.20, U$1.5
- removed net 37: C1.1, J1.19, U$1.6
- removed net 38: C2.1, J1.18, U$1.7
- removed net 39: C2.2, J1.17, U$1.8
- removed net 4: J2.8, U$1.24
- removed net N$13: C3.2, U$1.44, Y1.1
- removed net N$15: C4.2, U$1.43, Y1.3
- new net I2C_SCL_1: J2.4, R12.1, U$1.22
- new net I2C_SCL_A: J1.4, R10.1, U$1.15
- new net I2C_SDA_0: U$1.16
- new net I2C_SDA_1: J2.3, R11.1, U$1.24
- new net I2C_SDA_B: J1.3, R9.1
- new net N$11: JP1.1, R10.2
- new net N$4: JP3.3, R11.2
- new net N$5: JP3.1, R12.2
- new net N$6: JP1.3, R9.2
- new net XTAL_N_: C4.2, U$1.44, Y1.3
- new net XTAL_P_: C3.2, U$1.45, Y1.1
- net 0: now also R15.2; no longer J2.9
- net 3.3V: now also JP1.2, JP3.2, R15.1, U$1.37; no longer J1.5, J2.5, U$1.42, U$1.45
- net 32K_XN: no longer J1.15
- net 32K_XP: no longer J1.16
- net 5: no longer J2.12
- net CHIP_PU: no longer J1.6
- net FLASH_SHD: now also U$1.28; no longer U$1.29
- net FLASH_SWP: now also U$1.29; no longer U$1.28
- net GND: no longer J1.4, J2.4
- net U0RXD: now also U$1.41; no longer J2.16, U$1.37
- net U0TXD: now also U$1.42; no longer J2.15, U$1.36
- net VIN: now also J1.2, J2.2
- net VUSB: no longer J1.2, J2.2
- net V_BATT: no longer J1.3, J2.3
Routing:
- net I2C_SCL_1: track 0.00 -> 29.7 mm, vias 0 -> 2
- net I2C_SDA_1: track 0.00 -> 29.4 mm, vias 0 -> 1
- net VUSB: track 35.5 -> 6.65 mm
- net 16: track 27.0 -> 0.00 mm, vias 1 -> 0
- net V_BATT: track 40.3 -> 13.7 mm
- net VIN: track 10.9 -> 36.2 mm
- net 15: track 24.8 -> 0.00 mm, vias 1 -> 0
- net 17: track 24.0 -> 0.00 mm, vias 1 -> 0
- net 2: track 23.2 -> 0.00 mm, vias 1 -> 0
- net 3.3V: track 116.5 -> 139.7 mm
- net 4: track 22.6 -> 0.00 mm, vias 1 -> 0
- net 13: track 22.5 -> 0.00 mm, vias 1 -> 0
- net 12: track 22.1 -> 0.00 mm, vias 1 -> 0
- net 14: track 20.3 -> 0.00 mm, vias 1 -> 0
- net 19: track 19.9 -> 0.00 mm, vias 1 -> 0
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Other:
- board size 25.4 x 58.9 mm -> 27.9 x 58.9 mm
- board text added: "CHL A"
- board text added: "CHL B"
- board text added: "Director Board"
- board text added: "Spectacle!"
- board text removed: "!RST!"
- board text removed: "12"
- board text removed: "13"
- board text removed: "14"
- board text removed: "15"
- board text removed: "16"
- board text removed: "17"
- board text removed: "18"
- board text removed: "19"
- board text removed: "2"
- board text removed: "20"
- board text removed: "21"
- board text removed: "22"
- board text removed: "23"
- board text removed: "25"
- board text removed: "26"
- board text removed: "27"
- board text removed: "32"
- board text removed: "33"
- board text removed: "34"
- board text removed: "35"
- board text removed: "36"
- board text removed: "37"
- board text removed: "38"
- board text removed: "39"
- board text removed: "3V3"
- board text removed: "4"
- board text removed: "5"
- board text removed: "ESP32 Thing"
- board text removed: "GND"
- board text removed: "RX"
- board text removed: "TX"
- board text removed: "VBAT"
- board text removed: "VUSB"
