File: Hardware/esp32-thing.sch (EAGLE design)
At the start: 67 parts, among them Q1 2.5A/30V, Q2 MBT3904DW1T1, U1 MCP73831, U3 AP2112K-3.3V, U4 FT231XS, U5 W25Q32FVSS, Y1 26MHz, Y2 32.768kHz

Commit message: Incorporate changes from Jim's protos.
Parts:
- removed C1, C2: 270pF, SparkFun-Capacitors:CAP0603-CAP
- removed U2: (no value), esp32-thing-temp:ESP31B
- added JP1, JP3: (no value), SparkFun-Passives:JUMPER-PAD-3-NC_BY_TRACE
- added R10, R11, R12, R9: 4.7K, SparkFun-Resistors:4.7KOHM-1/10W-1%(0603)
- added R15: 10K, SparkFun-Resistors:10KOHM1/10W1%(0603)0603
- added U$1: ESP32, esp32-thing-temp:ESP32
- J1, J2: device SparkFun-Connectors:M20NOSILK -> SparkFun-Connectors:M04POLAR_LOCK
Connections:
- net N$11 renamed VCC_FLASH
- removed net 12: J1.8, U2.(GPIO12/ADC2:5/TOUCH5/RTC15/SPIQ)MTDI
- removed net 13: J1.7, U2.(GPIO13/ADC2:4/TOUCH4/RTC14/SPID/U0CTS)MTCK
- removed net 14: J1.9, U2.(GPIO14/ADC2:6/TOUCH6/RTC16/SPICLK)MTMS
- removed net 15: J2.11, U2.(GPIO15/ADC2:3/TOUCH3/RTC13/SPICSO/U0RTS)MTDO
- removed net 16: J2.6, U2.(HS1_DATA4)GPIO16
- removed net 17: J2.7, U2.(HS1_DATA5)GPIO17
- removed net 18: J2.13, U2.(VSPICLK/HS1_DATA7)GPIO18
- removed net 19: J2.20, U2.(VSPIQ/HS2_DATA2)GPIO19
- removed net 2: J2.10, U2.(ADC2:2/TOUCH2/RTC12/SPIWP)GPIO2
- removed net 20: J2.19, U2.(VSPID/HS2_DATA3)GPIO20
- removed net 21: J2.18, U2.(VSPIHD/HS2_CMD)GPIO21
- removed net 22: J2.17, U2.(VSPIWP/HS2_CLK)GPIO22
- removed net 23: J2.14
- removed net 25: J1.12, U2.(DAC1/ADC2:8/RTC6)GPIO25
- removed net 26: J1.11, U2.(DAC2/ADC2:9/RTC7)GPIO26
- removed net 27: J1.10, U2.(ADC2:7/TOUCH7/RTC17)GPIO27
- removed net 34: J1.14, U2.VDET_1(GPI34/ADC1:6)
- removed net 35: J1.13, U2.VDET_2(GPI35/ADC1:7)
- removed net 36: C1.2, J1.20, U2.SENSOR_VP(GPI36/ADC1:0/RTC0)
- removed net 37: C1.1, J1.19, U2.SENSOR_CAPP(GPI37/ADC1:1/RTC1)
- removed net 38: C2.1, J1.18, U2.SENSOR_CAPN(GPI38/ADC1:2/RTC2)
- removed net 39: C2.2, J1.17, U2.SENSOR_VN(GPI39/ADC1:3/RTC3)
- removed net 4: J2.8, U2.(ADC2:0/TOUCH0/RTC10/SPIHD)GPIO4
- removed net N$13: C3.2, U2.XTAL_P, Y1.1
- removed net N$15: C4.2, U2.XTAL_N, Y1.2
- new net I2C_SCL_1: J2.4, R12.1, U$1.(ADC2:2/TOUCH2/RTC12/SPIWP)GPIO2
- new net I2C_SCL_A: J1.4, R10.1, U$1.(DAC2/ADC2:9/RTC7)GPIO26
- new net I2C_SDA_0: U$1.(ADC2:7/TOUCH7/RTC17)GPIO27
- new net I2C_SDA_1: J2.3, R11.1, U$1.(ADC2:0/TOUCH0/RTC10/SPIHD)GPIO4
- new net I2C_SDA_B: J1.3, R9.1
- new net N$11: JP1.1, R10.2
- new net N$4: JP3.3, R11.2
- new net N$5: JP3.1, R12.2
- new net N$6: JP1.3, R9.2
- new net XTAL_N_: C4.2, U$1.XTAL_N, Y1.2
- new net XTAL_P_: C3.2, U$1.XTAL_P, Y1.1
- net 0: now also R15.2, U$1.(ADC2:1/TOUCH1/RTC11/CLK_OUT1)GPIO0; no longer J2.9, U2.(ADC2:1/TOUCH1/RTC11/CLK_OUT1)GPIO0
- net 3.3V: now also JP1.2, JP3.2, R15.1, U$1.VDD3P3_CPU, U$1.VDD3P3_RTC, U$1.VDDA, U$1.VDDA3P3; no longer J1.5, J2.5, U2.VDD3P3_CPU, U2.VDD3P3_RTC, U2.VDDA, U2.VDDA2, U2.VDDA3P3
- net 32K_XN: now also U$1.32K_XN(GPIO33/ADC1:5/TOUCH8/RTC8); no longer J1.15, U2.32K_XN(GPIO33/ADC1:5/TOUCH8/RTC8)
- net 32K_XP: now also U$1.32K_XP(GPIO32/ADC1:4/TOUCH9/RTC9); no longer J1.16, U2.32K_XP(GPIO32/ADC1:4/TOUCH9/RTC9)
- net 5: now also U$1.(VSPICS0/HS1_DATA6)GPIO5; no longer J2.12, U2.(VSPICS0/HS1_DATA6)GPIO5
- net CAP_10N: now also U$1.CAP_10N; no longer U2.CAP_10N
- net CHIP_PU: now also U$1.CHIP_PU; no longer J1.6, U2.CHIP_PU
- net FLASH_SCK: now also U$1.(GPIO6/SPICLK/HS1_CLK/U1CTS)SD_CLK; no longer U2.(GPIO6/SPICLK/HS1_CLK/U1CTS)SD_CLK
- net FLASH_SCS: now also U$1.(GPIO11/SPICSO/HS1_CMD/U1RTS)SD_CMD; no longer U2.(GPIO11/SPICSO/HS1_CMD/U1RTS)SD_CMD
- net FLASH_SDI: now also U$1.(GPIO8/SPID/HS1_DATA1)SD_DATA1; no longer U2.(GPIO8/SPID/HS1_DATA1)SD_DATA1
- net FLASH_SDO: now also U$1.(GPIO7/SPI1/HS1_DATA0)SD_DATA0; no longer U2.(GPIO7/SPI1/HS1_DATA0)SD_DATA0
- net FLASH_SHD: now also U$1.(GPIO9/SPIHD/HS1_DATA2/U1RX)SD_DATA2; no longer U2.(GPIO10/SPIWP/HS1_DATA3/U1TX)SD_DATA3
- net FLASH_SWP: now also U$1.(GPIO10/SPIWP/HS1_DATA3/U1TX)SD_DATA3; no longer U2.(GPIO9/SPIHD/HS1_DATA2/U1RX)SD_DATA2
- net FLASH_VDD: now also U$1.VDD3P3_SDIO; no longer U2.VDD3P3_SDIO
- net GND: now also U$1.GND; no longer J1.4, J2.4, U2.GND
- net LNA_IN: now also U$1.LNA_IN; no longer U2.LNA_IN
- net RES_14K: now also U$1.RES_14K; no longer U2.RES_14K
- net U0RXD: now also U$1.(GPIO3/CLK_OUT2/HS2_DATA0)U0RXD; no longer J2.16, U2.(GPIO3/CLK_OUT2/HS2_DATA0)U0RXD
- net U0TXD: now also U$1.(GPIO1/CLK_OUT3/HS2_DATA1)U0TXD; no longer J2.15, U2.(GPIO1/CLK_OUT3/HS2_DATA1)U0TXD
- net VIN: now also J1.2, J2.2
- net VUSB: no longer J1.2, J2.2
- net V_BATT: no longer J1.3, J2.3
Other:
- moved on the sheet: R1, S1, S2
