File: Hardware/Spectacle_Director_Board.sch (EAGLE design)
At the start: 72 parts, among them Q1 2.5A/30V, Q2 MBT3904DW1T1, U1 MCP73831, U3 AP2112K-3.3V, U4 FT231XS, U5 W25Q32FVSS, Y1 26MHz, Y2 32.768kHz

Commit message: Initial commit of finished layout
Parts:
- removed C14, C16: 0.1uF, SparkFun-Capacitors:0.1UF-25V(+80/-20%)(0603)
- removed C15, C19: 4.7uF, SparkFun-Capacitors:4.7UF-6.3V-10%(0603)0603
- removed J2: (no value), SparkFun-Connectors:M04POLAR_LOCK
- removed JP3: (no value), SparkFun-Passives:JUMPER-PAD-3-NC_BY_TRACE
- removed Q1: 2.5A/30V, SparkFun-DiscreteSemi:MOSFET-PCHANNELDMG2307L
- removed R10, R11, R12: 4.7K, SparkFun-Resistors:4.7KOHM-1/10W-1%(0603)
- removed R13, R14: 27, SparkFun-Resistors:27OHM1/10W1%(0603)0603-RES
- removed R7: 10K, SparkFun-Resistors:10KOHM1/10W1%(0603)0603
- removed SJ1, SJ2: JUMPER-PAD-2-NC_BY_TRACE, SparkFun-Passives:JUMPER-PAD-2-NC_BY_TRACE
- removed SJ3: JUMPER-PAD-3-2OF3_NC_BY_TRACE_SMALL, SparkFun-Passives:JUMPER-PAD-3-2OF3_NC_BY_TRACE_SMALL
- removed U4: FT231XS, SparkFun-DigitalIC:FT231XS
- added C2: 1.0uF, SparkFun-Capacitors:1.0UF-16V-10%(0603)
- added D5: PESD1CAN, SparkFun-DiscreteSemi:PESD1CAN
- added FD1, FD2, FD3, FD4: FIDUCIALUFIDUCIAL, SparkFun-Aesthetics:FIDUCIALUFIDUCIAL
- added H1, H2, H3, H4: STAND-OFF, SparkFun-Electromechanical:STAND-OFF
- added J4: AUDIO-JACK3, SparkFun-Connectors:AUDIO-JACK3
- added U$2: FOUR_LAYER_WARNING, SparkFun-Aesthetics:FOUR_LAYER_WARNING
- C11: value 0.1uF -> 4.7uF; device SparkFun-Capacitors:0.1UF-25V(+80/-20%)(0603) -> SparkFun-Capacitors:4.7UF-16V-20%,+80%-(1206)
- C12: value 47pF -> 0.1uF; device SparkFun-Capacitors:47PF-50V-5%(0603) -> SparkFun-Capacitors:0.1UF-25V-5%(0603)
- C13: value 47pF -> 4.7uF; device SparkFun-Capacitors:47PF-50V-5%(0603) -> SparkFun-Capacitors:4.7UF-16V-20%,+80%-(1206)
- C18, C20, C21, C23, C25: device SparkFun-Capacitors:0.1UF-25V(+80/-20%)(0603) -> SparkFun-Capacitors:0.1UF-16V(+-10%)(0402)
- C6: value 4.7uF -> 0.1uF; device SparkFun-Capacitors:4.7UF-6.3V-10%(0603)0603 -> SparkFun-Capacitors:0.1UF-25V-5%(0603)
- D1: value Yellow -> PESD1CAN; device SparkFun-LED:LED-YELLOW0603 -> SparkFun-DiscreteSemi:PESD1CAN
- D2: value BAT20J -> PESD1CAN; device SparkFun-DiscreteSemi:DIODE-SCHOTTKY-BAT20J -> SparkFun-DiscreteSemi:PESD1CAN
- J1: value (none) -> AUDIO-JACK3; device SparkFun-Connectors:M04POLAR_LOCK -> SparkFun-Connectors:AUDIO-JACK3
- JP1: value (none) -> JUMPER-PAD-3-NC_BY_PASTE; device SparkFun-Passives:JUMPER-PAD-3-NC_BY_TRACE -> SparkFun-Passives:JUMPER-PAD-3-NC_BY_PASTE
- JP2: value LiPo -> JUMPER-PAD-3-NC_BY_PASTE; device SparkFun-Connectors:M02JST-PTH-2 -> SparkFun-Passives:JUMPER-PAD-3-NC_BY_PASTE
- R3: value 1K -> 2.2k; device SparkFun-Resistors:1KOHM-1/10W-1%(0603) -> SparkFun-Resistors:2.2KOHM-1/10W-1%(0603)
- R5: value DNP -> 2.2k; device SparkFun-Passives:RESISTORPTH-1/6W -> SparkFun-Resistors:2.2KOHM-1/10W-1%(0603)
- R6: value 2.0k -> 2.2k; device SparkFun-Resistors:2.0KOHM1/10W5%(0603) -> SparkFun-Resistors:2.2KOHM-1/10W-1%(0603)
- R9: value 4.7K -> 2.2k; device SparkFun-Resistors:4.7KOHM-1/10W-1%(0603) -> SparkFun-Resistors:2.2KOHM-1/10W-1%(0603)
- S1, S2: device SparkFun-Electromechanical:SWITCH-MOMENTARY-2SMD-4.6X2.8MM -> SparkFun-Electromechanical:SWITCH_SPST_4_PINRECT
- U1: value MCP73831 -> CY7C65213; device SparkFun-PowerIC:MCP73831 -> SparkFun-DigitalIC:CY7C65213
Connections:
- removed net 3.3V_F: C16.1, U4.!RESET, U4.3V3OUT, U4.VCCIO
- removed net D+: C13.1, JP15.D+, R14.1
- removed net D-: C12.1, JP15.D-, R13.1
- removed net I2C_SCL_A: J1.4, R10.1, U$1.(DAC2/ADC2:9/RTC7)GPIO26
- removed net I2C_SDA_B: J1.3, R9.1
- removed net N$11: JP1.1, R10.2
- removed net N$14: R5.2, SJ1.2, U1.PROG
- removed net N$16: R6.2, SJ1.1
- removed net N$17: D1.A, R3.2
- removed net N$9: D1.C, U1.STAT
- removed net VCC_FLASH: C17.1, SJ3.2, U5.VCC
- removed net VIN: C7.1, D2.C, J1.2, J2.2, Q1.S, U3.EN, U3.IN
- removed net V_BATT: C6.1, JP2.2, Q1.D, U1.VBAT
- new net I2C_SCL_0: D5.1, J1.RING2, R6.1, U$1.(DAC2/ADC2:9/RTC7)GPIO26
- new net VDD: C2.1, U1.VCCD
- net 0: now also S2.3; no longer S2.2
- net 3.3V: now also C12.1, C13.1, C17.1, JP2.2, R4.1, U1.VCCIO, U5.VCC; no longer JP3.2, SJ2.2, SJ3.3
- net CHIP_PU: now also S1.3; no longer S1.2
- net DTR: now also U1.DTR; no longer U4.!DTR
- net FLASH_VDD: no longer SJ3.1
- net GND: now also C2.2, D1.3, D2.3, D5.3, J1.TIP, J4.TIP; no longer C14.2, C15.2, C16.2, C19.2, J1.1, J2.1, JP2.1, R5.1, R6.1, R7.1, U1.VSS, U4.GND@16, U4.GND@6
- net I2C_SCL_1: now also D1.1, J4.RING2, R3.1; no longer J2.4, R12.1
- net I2C_SDA_0: now also D5.2, J1.RING1, R9.1
- net I2C_SDA_1: now also D1.2, J4.RING1, R5.1; no longer J2.3, R11.1
- net N$3: now also JP1.3, R3.2; no longer R4.1, SJ2.1
- net N$4: now also JP2.3, R6.2; no longer JP3.3, R11.2
- net N$5: now also JP2.1, R9.2; no longer JP3.1, R12.2
- net N$6: now also JP1.1, R5.2; no longer JP1.3, R9.2
- net N$7: now also JP15.D-, U1.USBDM; no longer R13.2, U4.USBDM
- net N$8: now also JP15.D+, U1.USBDP; no longer R14.2, U4.USBDP
- net RTS: now also U1.CTS; no longer U4.!RTS
- net U0RXD: no longer U4.TXD
- net U0TXD: now also U1.RXD; no longer U4.RXD
- net VUSB: no longer C11.1
- net V_USB: now also C11.1, C6.1, C7.1, D2.1, J1.EARTH, J4.EARTH, U1.VCC, U3.EN, U3.IN; no longer C14.1, C15.1, C19.1, D2.A, Q1.G, R3.1, R7.2, U1.VIN, U4.VCC
Other:
- note added: "C12 and C13 to be near U1.4"
- note added: "C2 to be near U1.17"
- note added: "C6 and C11 to be near U1.20"
- note added: "CY7C65213 (USB-to-Serial Converter)"
- note added: "Output Jacks"
- note added: "Voltage Regulator"
- note removed: "Charge current: I_CHG = 1000 / R_PROG R_PROG=2k : I_CHG=500mA"
- note removed: "FT231XS (USB-to-Serial Converter)"
- note removed: "Headers"
- note removed: "Lithium-Polymer Battery Charger (1-cell)"
- note removed: "SJ1 can be cut to modify the charge- current programming resistor."
- note removed: "V_BATT should be a single- cell LiPo battery."
- note removed: "Voltage Regulator and Battery Charger"
- moved on the sheet: C11, C12, C13, C17, C26, C6, C9, D3, D4, F1, JP15, R1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

Commit message: For QC review
Parts:
- C26, C9: value (none) -> 22pF; device SparkFun-Passives:CAP0603-CAP -> SparkFun-Capacitors:22PF-50V-5%(0603)
- renumbered U$1 to U4
Other:
- note added: "Mike Hord"
- note removed: "Jim Lindblom"

Commit message: Feedback from QC review
Parts:
- R2: PROD_ID (none) -> RES-13340
Changed lines of the file:
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@@
 <part name="C4" library="SparkFun-Capacitors" deviceset="10PF-50V-5%(0603)" device="" value="10pF"/>
 <part name="C5" library="SparkFun-Capacitors" deviceset="10NF/10000PF-50V-10%(0603)" device="" value="10nF"/>
-<part name="R2" library="SparkFun-Passives" deviceset="RESISTOR" device="0603-RES" value="14k"/>
+<part name="R2" library="SparkFun-Passives" deviceset="RESISTOR" device="0603-RES" value="14k">
+<attribute name="PROD_ID" value="RES-13340"/>
+</part>
 <part name="GND3" library="SparkFun-Aesthetics" deviceset="GND" device=""/>
 <part name="GND35" library="SparkFun-Aesthetics" deviceset="GND" device=""/>
@@
 <instance part="C4" gate="G$1" x="50.8" y="124.46" rot="MR270"/>
 <instance part="C5" gate="G$1" x="60.96" y="78.74" rot="R180"/>
-<instance part="R2" gate="G$1" x="66.04" y="76.2" rot="R90"/>
+<instance part="R2" gate="G$1" x="66.04" y="76.2" rot="R90">
+<attribute name="PROD_ID" x="66.04" y="76.2" size="1.778" layer="96" rot="R90" display="off"/>
+</instance>
 <instance part="GND3" gate="1" x="71.12" y="63.5"/>
 <instance part="GND35" gate="1" x="238.76" y="154.94" rot="MR0"/>

Commit message: Changes due to Espressif changing chip before release
Parts:
- removed U4: ESP32, esp32-thing-temp:ESP32
- added C1: 3.0nF, esp32-thing-temp:3.0NF-0603-50V-5%
- added R7: 10K, SparkFun-Resistors:10KOHM-1/10W-1%(0603)0603
- added U2: ESP3212, esp32-thing-temp:ESP3212
- R2: value 14k -> 20k; device SparkFun-Passives:RESISTOR0603-RES -> SparkFun-Resistors:20KOHM1/10W1%(0603); PROD_ID RES-13340 -> (none)
Connections:
- removed net RES_14K: R2.2, U4.RES_14K
- new net N$11: C1.2, R2.2, U2.CAP2
- net 0: now also R7.1, U2.(ADC2:1/TOUCH1/RTC11/CLK_OUT1)GPIO0; no longer U4.(ADC2:1/TOUCH1/RTC11/CLK_OUT1)GPIO0
- net 3.3V: now also R7.2, U2.VDD3P3_CPU, U2.VDD3P3_RTC, U2.VDDA, U2.VDDA3P3; no longer U4.VDD3P3_CPU, U4.VDD3P3_RTC, U4.VDDA, U4.VDDA3P3
- net 32K_XN: now also U2.32K_XN(GPIO33/ADC1:5/TOUCH8/RTC8); no longer U4.32K_XN(GPIO33/ADC1:5/TOUCH8/RTC8)
- net 32K_XP: now also U2.32K_XP(GPIO32/ADC1:4/TOUCH9/RTC9); no longer U4.32K_XP(GPIO32/ADC1:4/TOUCH9/RTC9)
- net 5: now also U2.(VSPICS0/HS1_DATA6)GPIO5; no longer U4.(VSPICS0/HS1_DATA6)GPIO5
- net CAP_10N: now also C1.1, R2.1, U2.CAP1; no longer U4.CAP_10N
- net CHIP_PU: now also U2.CHIP_PU; no longer U4.CHIP_PU
- net FLASH_SCK: now also U2.(GPIO6/SPICLK/HS1_CLK/U1CTS)SD_CLK; no longer U4.(GPIO6/SPICLK/HS1_CLK/U1CTS)SD_CLK
- net FLASH_SCS: now also U2.(GPIO11/SPICSO/HS1_CMD/U1RTS)SD_CMD; no longer U4.(GPIO11/SPICSO/HS1_CMD/U1RTS)SD_CMD
- net FLASH_SDI: now also U2.(GPIO8/SPID/HS1_DATA1)SD_DATA1; no longer U4.(GPIO8/SPID/HS1_DATA1)SD_DATA1
- net FLASH_SDO: now also U2.(GPIO7/SPI1/HS1_DATA0)SD_DATA0; no longer U4.(GPIO7/SPI1/HS1_DATA0)SD_DATA0
- net FLASH_SHD: now also U2.(GPIO9/SPIHD/HS1_DATA2/U1RX)SD_DATA2; no longer U4.(GPIO9/SPIHD/HS1_DATA2/U1RX)SD_DATA2
- net FLASH_SWP: now also U2.(GPIO10/SPIWP/HS1_DATA3/U1TX)SD_DATA3; no longer U4.(GPIO10/SPIWP/HS1_DATA3/U1TX)SD_DATA3
- net FLASH_VDD: now also U2.VDD3P3_SDIO; no longer U4.VDD3P3_SDIO
- net GND: now also U2.GND; no longer R2.1, U4.GND
- net I2C_SCL_0: now also U2.(DAC2/ADC2:9/RTC7)GPIO26; no longer U4.(DAC2/ADC2:9/RTC7)GPIO26
- net I2C_SCL_1: now also U2.(ADC2:2/TOUCH2/RTC12/SPIWP)GPIO2; no longer U4.(ADC2:2/TOUCH2/RTC12/SPIWP)GPIO2
- net I2C_SDA_0: now also U2.(ADC2:7/TOUCH7/RTC17)GPIO27; no longer U4.(ADC2:7/TOUCH7/RTC17)GPIO27
- net I2C_SDA_1: now also U2.(ADC2:0/TOUCH0/RTC10/SPIHD)GPIO4; no longer U4.(ADC2:0/TOUCH0/RTC10/SPIHD)GPIO4
- net LNA_IN: now also U2.LNA_IN; no longer U4.LNA_IN
- net U0RXD: now also U2.(GPIO3/CLK_OUT2/HS2_DATA0)U0RXD; no longer U4.(GPIO3/CLK_OUT2/HS2_DATA0)U0RXD
- net U0TXD: now also U2.(GPIO1/CLK_OUT3/HS2_DATA1)U0TXD; no longer U4.(GPIO1/CLK_OUT3/HS2_DATA1)U0TXD
- net XTAL_N_: now also U2.XTAL_N; no longer U4.XTAL_N
- net XTAL_P_: now also U2.XTAL_P; no longer U4.XTAL_P
Other:
- moved on the sheet: C5, R2, S2

Commit message: Changes from design review for v02
Parts:
- removed R15: 10K, SparkFun-Resistors:10KOHM1/10W1%(0603)0603
- added C14: 1.0uF, SparkFun-Capacitors:1.0UF-16V-10%(0603)
Connections:
- net 0: no longer R15.2
- net 3.3V: now also C14.1; no longer R15.1
- net GND: now also C14.2
- net U0RXD: now also U1.TXD
Other:
- note added: "JP1 and JP2 disable I2C pull-up resistors"
- note added: "v02"
- note removed: "v01"
- moved on the sheet: U1
Changed lines of the file:
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@@
 <part name="GND37" library="SparkFun-Aesthetics" deviceset="GND" device=""/>
 <part name="LOGO2" library="SparkFun-Aesthetics" deviceset="OSHW-LOGO" device="MINI" value="OSHW-LOGOMINI"/>
-<part name="R15" library="SparkFun-Resistors" deviceset="10KOHM1/10W1%(0603)" device="0603" value="10K"/>
-<part name="SUPPLY5" library="SparkFun-Aesthetics" deviceset="3.3V" device=""/>
 <part name="U1" library="SparkFun-DigitalIC" deviceset="CY7C65213" device=""/>
 <part name="C2" library="SparkFun-Capacitors" deviceset="1.0UF-16V-10%(0603)" device="" value="1.0uF"/>
@@
 <part name="R7" library="SparkFun-Resistors" deviceset="10KOHM-1/10W-1%(0603)" device="0603" value="10K"/>
 <part name="SUPPLY25" library="SparkFun-Aesthetics" deviceset="3.3V" device=""/>
+<part name="C14" library="SparkFun-Capacitors" deviceset="1.0UF-16V-10%(0603)" device="" value="1.0uF"/>
+<part name="GND13" library="SparkFun-Aesthetics" deviceset="GND" device=""/>
+<part name="SUPPLY5" library="SparkFun-Aesthetics" deviceset="3.3V" device=""/>
 </parts>
 <sheets>
@@
 <text x="261.62" y="137.16" size="2.54" layer="97" align="top-left">GPIO5 LED</text>
 <text x="200.66" y="104.14" size="2.54" layer="97" align="top-left">Output Jacks</text>
-<text x="421.64" y="10.16" size="2.54" layer="94" align="top-left">v01</text>
+<text x="421.64" y="10.16" size="2.54" layer="94" align="top-left">v02</text>
 <text x="355.6" y="10.16" size="2.54" layer="94" align="top-left">Mike Hord</text>
 <wire x1="431.8" y1="66.04" x2="330.2" y2="66.04" width="0.2032" layer="97" style="longdash"/>
@@
 near U1.17</text>
 <wire x1="259.08" y1="106.68" x2="330.2" y2="106.68" width="0.2032" layer="97" style="longdash"/>
+<text x="254" y="91.44" size="1.778" layer="97">JP1 and JP2 disable
+I2C pull-up resistors</text>
 </plain>
 <instances>
@@
 <instance part="GND37" gate="1" x="307.34" y="114.3"/>
 <instance part="LOGO2" gate="G$1" x="182.88" y="10.16"/>
-<instance part="R15" gate="G$1" x="347.98" y="127" rot="R270"/>
-<instance part="SUPPLY5" gate="G$1" x="347.98" y="134.62"/>
-<instance part="U1" gate="G$1" x="363.22" y="213.36"/>
+<instance part="U1" gate="G$1" x="365.76" y="213.36"/>
 <instance part="C2" gate="G$1" x="172.72" y="238.76"/>
 <instance part="SUPPLY17" gate="VDD" x="172.72" y="251.46"/>
@@
 <instance part="R7" gate="G$1" x="373.38" y="53.34" rot="R90"/>
 <instance part="SUPPLY25" gate="G$1" x="373.38" y="60.96"/>
+<instance part="C14" gate="G$1" x="30.48" y="22.86"/>
+<instance part="GND13" gate="1" x="30.48" y="15.24"/>
+<instance part="SUPPLY5" gate="G$1" x="30.48" y="30.48"/>
 </instances>
 <busses>
@@
 </segment>
 <segment>
-<pinref part="SUPPLY5" gate="G$1" pin="3.3V"/>
-<pinref part="R15" gate="G$1" pin="1"/>
-<wire x1="347.98" y1="134.62" x2="347.98" y2="132.08" width="0.1524" layer="91"/>
-</segment>
-<segment>
 <pinref part="C12" gate="G$1" pin="1"/>
 <wire x1="208.28" y1="243.84" x2="208.28" y2="248.92" width="0.1524" layer="91"/>
@@
 <segment>
 <pinref part="U1" gate="G$1" pin="VCCIO"/>
-<wire x1="358.14" y1="241.3" x2="347.98" y2="241.3" width="0.1524" layer="91"/>
+<wire x1="360.68" y1="241.3" x2="347.98" y2="241.3" width="0.1524" layer="91"/>
 <wire x1="347.98" y1="241.3" x2="347.98" y2="266.7" width="0.1524" layer="91"/>
 <pinref part="SUPPLY20" gate="G$1" pin="3.3V"/>
@@
 <pinref part="R7" gate="G$1" pin="2"/>
 <wire x1="373.38" y1="60.96" x2="373.38" y2="58.42" width="0.1524" layer="91"/>
+</segment>
+<segment>
+<pinref part="C14" gate="G$1" pin="1"/>
+<wire x1="30.48" y1="27.94" x2="30.48" y2="30.48" width="0.1524" layer="91"/>
+<pinref part="SUPPLY5" gate="G$1" pin="3.3V"/>
 </segment>
 </net>
@@
 <wire x1="259.08" y1="35.56" x2="259.08" y2="33.02" width="0.1524" layer="91"/>
 </segment>
+<segment>
+<pinref part="C14" gate="G$1" pin="2"/>
+<pinref part="GND13" gate="1" pin="GND"/>
+<wire x1="30.48" y1="20.32" x2="30.48" y2="17.78" width="0.1524" layer="91"/>
+</segment>
 </net>
 <net name="LNA_IN" class="0">
@@
 <segment>
 <label x="393.7" y="254" size="1.27" layer="95" xref="yes"/>
-<wire x1="388.62" y1="254" x2="393.7" y2="254" width="0.1524" layer="91"/>
+<wire x1="391.16" y1="254" x2="393.7" y2="254" width="0.1524" layer="91"/>
+<pinref part="U1" gate="G$1" pin="TXD"/>
 </segment>
 </net>
@@
 <label x="393.7" y="251.46" size="1.27" layer="95" xref="yes"/>
 <pinref part="U1" gate="G$1" pin="RXD"/>
-<wire x1="388.62" y1="251.46" x2="393.7" y2="251.46" width="0.1524" layer="91"/>
+<wire x1="391.16" y1="251.46" x2="393.7" y2="251.46" width="0.1524" layer="91"/>
 </segment>
 </net>
@@
 <label x="393.7" y="241.3" size="1.27" layer="95" xref="yes"/>
 <pinref part="U1" gate="G$1" pin="DTR"/>
-<wire x1="388.62" y1="241.3" x2="393.7" y2="241.3" width="0.1524" layer="91"/>
+<wire x1="391.16" y1="241.3" x2="393.7" y2="241.3" width="0.1524" layer="91"/>
 </segment>
 <segment>
@@
 <segment>
 <pinref part="U1" gate="G$1" pin="VCC"/>
-<wire x1="358.14" y1="246.38" x2="355.6" y2="246.38" width="0.1524" layer="91"/>
+<wire x1="360.68" y1="246.38" x2="355.6" y2="246.38" width="0.1524" layer="91"/>
 <pinref part="SUPPLY21" gate="G$1" pin="V_USB"/>
 <wire x1="355.6" y1="269.24" x2="355.6" y2="246.38" width="0.1524" layer="91"/>
@@
 <label x="393.7" y="246.38" size="1.27" layer="95" xref="yes"/>
 <pinref part="U1" gate="G$1" pin="CTS"/>
-<wire x1="388.62" y1="246.38" x2="393.7" y2="246.38" width="0.1524" layer="91"/>
+<wire x1="391.16" y1="246.38" x2="393.7" y2="246.38" width="0.1524" layer="91"/>
 </segment>
 <segment>
@@
 <net name="0" class="0">
 <segment>
-<wire x1="375.92" y1="114.3" x2="347.98" y2="114.3" width="0.1524" layer="91"/>
+<wire x1="375.92" y1="114.3" x2="342.9" y2="114.3" width="0.1524" layer="91"/>
 <label x="342.9" y="114.3" size="1.27" layer="95" rot="R180" xref="yes"/>
 <pinref part="Q2" gate="Q2" pin="C"/>
-<wire x1="347.98" y1="114.3" x2="342.9" y2="114.3" width="0.1524" layer="91"/>
 <wire x1="375.92" y1="114.3" x2="375.92" y2="116.84" width="0.1524" layer="91"/>
-<pinref part="R15" gate="G$1" pin="2"/>
-<wire x1="347.98" y1="121.92" x2="347.98" y2="114.3" width="0.1524" layer="91"/>
-<junction x="347.98" y="114.3"/>
 </segment>
 <segment>
@@
 <segment>
 <pinref part="U1" gate="G$1" pin="VCCD"/>
-<wire x1="358.14" y1="243.84" x2="350.52" y2="243.84" width="0.1524" layer="91"/>
+<wire x1="360.68" y1="243.84" x2="350.52" y2="243.84" width="0.1524" layer="91"/>
 <wire x1="350.52" y1="243.84" x2="350.52" y2="261.62" width="0.1524" layer="91"/>
 <pinref part="SUPPLY7" gate="VDD" pin="VDD"/>
@@
 <pinref part="JP15" gate="G$1" pin="D-"/>
 <pinref part="U1" gate="G$1" pin="USBDM"/>
-<wire x1="284.48" y1="254" x2="358.14" y2="254" width="0.1524" layer="91"/>
+<wire x1="284.48" y1="254" x2="360.68" y2="254" width="0.1524" layer="91"/>
 </segment>
 </net>
@@
 <pinref part="JP15" gate="G$1" pin="D+"/>
 <pinref part="U1" gate="G$1" pin="USBDP"/>
-<wire x1="284.48" y1="251.46" x2="358.14" y2="251.46" width="0.1524" layer="91"/>
-</segment>
-</net>
+<wire x1="284.48" y1="251.46" x2="360.68" y2="251.46" width="0.1524" layer="91"/>
+</segment>
+</net>
